File: USB-Relay-Board.kicad_pcb (KiCad board)
At the start: 2 copper layers, 27 parts, among them J1 USB_B, J2 Conn_01x12, J3 Conn_01x12, U1 STM32F070F6Px, U2 TLV70036_SOT23-5, U3 ULN2804A, Y1 Crystal

Commit message: Auto commit: Changes detected on 2024-10-23 06:04:16
Parts:
- moved C12 25.3 mm to (86.0, 76.0)
- moved C7 24.6 mm to (102.5, 53.0), turned to 0 degrees
- moved C6 19.9 mm to (102.5, 56.0), turned to 0 degrees
- moved C9 17.5 mm to (87.0, 65.0), turned to 180 degrees
- moved C3 17.1 mm to (102.6, 68.0), turned to 0 degrees
- moved C10 17.1 mm to (87.1, 62.0), turned to 180 degrees
- moved C5 16.2 mm to (102.5, 59.0), turned to 0 degrees
- moved C4 14.4 mm to (102.5, 65.0), turned to 0 degrees
- moved C8 14.1 mm to (102.5, 62.0), turned to 0 degrees
- moved C11 9.46 mm to (103.0, 74.0), turned to 90 degrees
- moved Y1 3.82 mm to (97.0, 74.5), turned to 180 degrees
- moved U1 3.02 mm to (94.5, 62.0), turned to 180 degrees
Routing:
- net +3.3V: track 0.46 -> 26.0 mm
- net Net-(U1-PF1): track 0.00 -> 20.5 mm
- net Net-(U1-PF0): track 0.00 -> 18.8 mm
Other:
- board text removed: "EUGENIA <3"

Commit message: Auto commit: Changes detected on 2024-10-23 06:16:01
Routing:
- net Net-(U1-PF1): track 20.5 -> 6.32 mm
Changed lines of the file:
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@@
 		(tags "capacitor handsolder")
 		(property "Reference" "C3"
-			(at 0 -1.68 360)
+			(at 0 -1.68 0)
 			(layer "F.SilkS")
 			(effects
@@
 		)
 		(property "Value" "100nF"
-			(at 0 1.68 360)
+			(at 0 1.68 0)
 			(layer "F.Fab")
 			(effects
@@
 		)
 		(fp_text user "${REFERENCE}"
-			(at 0 0 360)
+			(at 0 0 0)
 			(layer "F.Fab")
 			(effects
@@
 		(tags "capacitor handsolder")
 		(property "Reference" "C10"
-			(at 0 -1.68 360)
+			(at 0 -1.68 0)
 			(layer "F.SilkS")
 			(effects
@@
 		)
 		(property "Value" "1uF"
-			(at 0 1.68 360)
+			(at 0 1.68 0)
 			(layer "F.Fab")
 			(effects
@@
 		)
 		(fp_text user "${REFERENCE}"
-			(at 0 0 360)
+			(at 0 0 0)
 			(layer "F.Fab")
 			(effects
@@
 		(tags "capacitor handsolder")
 		(property "Reference" "C9"
-			(at 0 -1.68 360)
+			(at 0 -1.68 0)
 			(layer "F.SilkS")
 			(effects
@@
 		)
 		(property "Value" "10nF"
-			(at 0 1.68 360)
+			(at 0 1.68 0)
 			(layer "F.Fab")
 			(effects
@@
 		)
 		(fp_text user "${REFERENCE}"
-			(at 0 0 360)
+			(at 0 0 0)
 			(layer "F.Fab")
 			(effects
@@
 		(tags "capacitor handsolder")
 		(property "Reference" "C8"
-			(at 0 -1.68 360)
+			(at 0 -1.68 0)
 			(layer "F.SilkS")
 			(effects
@@
 		)
 		(property "Value" "4.7nF"
-			(at 0 1.68 360)
+			(at 0 1.68 0)
 			(layer "F.Fab")
 			(effects
@@
 		)
 		(fp_text user "${REFERENCE}"
-			(at 0 0 360)
+			(at 0 0 0)
 			(layer "F.Fab")
 			(effects
@@
 		(tags "capacitor handsolder")
 		(property "Reference" "C5"
-			(at 0 -1.68 360)
+			(at 0 -1.68 0)
 			(layer "F.SilkS")
 			(effects
@@
 		)
 		(property "Value" "100nF"
-			(at 0 1.68 360)
+			(at 0 1.68 0)
 			(layer "F.Fab")
 			(effects
@@
 		)
 		(fp_text user "${REFERENCE}"
-			(at 0 0 360)
+			(at 0 0 0)
 			(layer "F.Fab")
 			(effects
@@
 		(tags "capacitor handsolder")
 		(property "Reference" "C6"
-			(at 0 -1.68 360)
+			(at 0 -1.68 0)
 			(layer "F.SilkS")
 			(effects
@@
 		)
 		(property "Value" "100nF"
-			(at 0 1.68 360)
+			(at 0 1.68 0)
 			(layer "F.Fab")
 			(effects
@@
 		)
 		(fp_text user "${REFERENCE}"
-			(at 0 0 360)
+			(at 0 0 0)
 			(layer "F.Fab")
 			(effects
@@
 		)
 		(property "Value" "Crystal"
-			(at 2.45 3.525 360)
+			(at 2.45 3.525 0)
 			(layer "F.Fab")
 			(hide yes)
@@
 		(tags "capacitor handsolder")
 		(property "Reference" "C7"
-			(at 0 -1.68 360)
+			(at 0 -1.68 0)
 			(layer "F.SilkS")
 			(effects
@@
 		)
 		(property "Value" "100nF"
-			(at 0 1.68 360)
+			(at 0 1.68 0)
 			(layer "F.Fab")
 			(effects
@@
 		)
 		(fp_text user "${REFERENCE}"
-			(at 0 0 360)
+			(at 0 0 0)
 			(layer "F.Fab")
 			(effects
@@
 		(tags "TSSOP SO")
 		(property "Reference" "U1"
-			(at 0 -4.2 360)
+			(at 0 -4.2 0)
 			(layer "F.SilkS")
 			(effects
@@
 		)
 		(property "Value" "STM32F070F6Px"
-			(at 2 4.2 360)
+			(at 2 4.2 0)
 			(layer "F.Fab")
 			(hide yes)
@@
 		)
 		(fp_text user "${REFERENCE}"
-			(at 0 0 360)
+			(at 0 0 0)
 			(layer "F.Fab")
 			(effects
@@
 		(tags "capacitor handsolder")
 		(property "Reference" "C4"
-			(at 0 -1.68 360)
+			(at 0 -1.68 0)
 			(layer "F.SilkS")
 			(effects
@@
 		)
 		(property "Value" "100nF"
-			(at 0 1.68 360)
+			(at 0 1.68 0)
 			(layer "F.Fab")
 			(effects
@@
 		)
 		(fp_text user "${REFERENCE}"
-			(at 0 0 360)
+			(at 0 0 0)
 			(layer "F.Fab")
 			(effects
@@
 	)
 	(segment
-		(start 95 65.287501)
-		(end 95 64)
-		(width 0.2)
-		(layer "F.Cu")
-		(net 5)
-	)
-	(segment
 		(start 86 74.9625)
 		(end 91.6375 74.9625)
 		(width 0.2)
 		(layer "F.Cu")
-		(net 5)
-	)
-	(segment
-		(start 95.375 63.625)
-		(end 97.4 63.625)
-		(width 0.2)
-		(layer "F.Cu")
-		(net 5)
-	)
-	(segment
-		(start 92.11875 74.48125)
-		(end 92.11875 68.168751)
-		(width 0.2)
-		(layer "F.Cu")
-		(net 5)
-	)
-	(segment
-		(start 92.11875 68.168751)
-		(end 95 65.287501)
-		(width 0.2)
-		(layer "F.Cu")
-		(net 5)
-	)
-	(segment
-		(start 95 64)
-		(end 95.375 63.625)
-		(width 0.2)
-		(layer "F.Cu")

Commit message: Auto commit: Changes detected on 2024-10-23 06:18:03
Routing:
- net +3.3V: track 26.0 -> 19.8 mm
Changed lines of the file:
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@@
-	)
-	(segment
-		(start 91.675 62.325)
-		(end 88.4625 62.325)
-		(width 0.2)
-		(layer "F.Cu")
-		(net 3)
 	)
 	(segment
@@
 		(width 0.2)
 		(layer "F.Cu")
-		(net 3)
-	)
-	(segment
-		(start 88.075 65)
-		(end 88.075 62.0625)
-		(width 0.2)
-		(layer "F.Cu")
